Commit message: gazebo added

File: quadruped_spider/spiderbot/urdf/spiderbot.xacro (robot description, xacro)
@@ -6,5 +6,5 @@
 	<!-- Include Robot's urdf filepath -->
 	<!-- Include Lidar's urdf filepath -->
-	<xacro:include filename="$(find spiderbot)/urdf/spiderbot.urdf"/>
+	<xacro:include filename="$(find spiderbot)/urdf/my_spider/spiderbotv8_.urdf"/>
 	<xacro:include filename="$(find spiderbot)/urdf/ydlidar.urdf"/>
 <!-- Add your gazebo sensors here -->

File: quadruped_spider/spiderbot/urdf/ydlidar.urdf (robot description, URDF)
Before this commit: robot ydlidar, 2 links, 1 joints
Links:
- link base_laser: mass 0.15717 -> 0.015717
- link laser_frame: mass 0.25482 -> 0.025482

Commit message: pid tunned

File: quadruped_spider/spiderbot/urdf/spiderbot.xacro (robot description, xacro)
@@ -152,5 +152,5 @@
 	</gazebo>
     <gazebo reference="front_right_link1">
-		<material>Gazebo/Green</material>
+		<material>Gazebo/Grey</material>
 	</gazebo>
     <gazebo reference="front_left_link0">
@@ -158,5 +158,5 @@
 	</gazebo>
     <gazebo reference="front_left_link1">
-		<material>Gazebo/Green</material>
+		<material>Gazebo/Grey</material>
 	</gazebo>
     <gazebo reference="rear_right_link0">
@@ -164,5 +164,5 @@
 	</gazebo>
     <gazebo reference="rear_right_link1">
-		<material>Gazebo/Green</material>
+		<material>Gazebo/Grey</material>
 	</gazebo>
     <gazebo reference="rear_left_link0">
@@ -170,5 +170,5 @@
 	</gazebo>
     <gazebo reference="rear_left_link1">
-		<material>Gazebo/Green</material>
+		<material>Gazebo/Grey</material>
 	</gazebo>
     <!--Dummy Link-->
