Commit message: urdf update

File: quadruped_spider/spiderbot/urdf/my_spider/spiderbotv8_.urdf (robot description, URDF)
Before this commit: robot spiderbot, 9 links, 8 joints
Joints:
- joint joint_front_left_link0: limit lower=-3.14 upper=3.14 effort=2 velocity=0.2 -> lower=-0.523599 upper=0.523599 effort=2 velocity=0.02
- joint joint_front_left_link1: limit lower=-3.14 upper=3.14 effort=2 velocity=0.2 -> lower=-0.523599 upper=0.523599 effort=2 velocity=0.02
- joint joint_front_right_link0: limit lower=-3.14 upper=3.14 effort=2 velocity=0.2 -> lower=-0.5236 upper=0.5236 effort=2 velocity=0.02
- joint joint_front_right_link1: limit lower=-3.14 upper=3.14 effort=2 velocity=0.2 -> lower=-0.523599 upper=0.523599 effort=2 velocity=0.02
- joint joint_rear_left_link0: limit lower=-3.14 upper=3.14 effort=2 velocity=0.2 -> lower=-0.523599 upper=0.523599 effort=2 velocity=0.02
- joint joint_rear_left_link1: limit lower=-3.14 upper=3.14 effort=2 velocity=0.2 -> lower=-0.523599 upper=0.523599 effort=2 velocity=0.02
- joint joint_rear_right_link0: limit lower=-3.14 upper=3.14 effort=2 velocity=0.2 -> lower=-0.523599 upper=0.523599 effort=2 velocity=0.02
- joint joint_rear_right_link1: limit lower=-3.14 upper=3.14 effort=2 velocity=0.2 -> lower=-0.5236 upper=0.5236 effort=2 velocity=0.02

Commit message: display.launch resolved

File: quadruped_spider/spiderbot/urdf/my_spider/spiderbotv8_.urdf (robot description, URDF)
Before this commit: robot spiderbot, 9 links, 8 joints
Links:
- link base_link: geometry collision mesh filename=package://spiderbot/meshes/my_spider/base_link.STL; visual mesh filename=package://spiderbot/meshes/my_spider/base_link.STL
- link front_left_link0: geometry collision mesh filename=package://spiderbot/meshes/my_spider/r1.STL; visual mesh filename=package://spiderbot/meshes/my_spider/r1.STL
- link front_left_link1: geometry collision mesh filename=package://spiderbot/meshes/my_spider/sr1.STL; visual mesh filename=package://spiderbot/meshes/my_spider/sr1.STL
- link front_right_link0: geometry collision mesh filename=package://spiderbot/meshes/my_spider/r1.STL; visual mesh filename=package://spiderbot/meshes/my_spider/r1.STL
- link front_right_link1: geometry collision mesh filename=package://spiderbot/meshes/my_spider/sr1.STL; visual mesh filename=package://spiderbot/meshes/my_spider/sr1.STL
- link rear_left_link0: geometry collision mesh filename=package://spiderbot/meshes/my_spider/r1.STL; visual mesh filename=package://spiderbot/meshes/my_spider/r1.STL
- link rear_left_link1: geometry collision mesh filename=package://spiderbot/meshes/my_spider/sr1.STL; visual mesh filename=package://spiderbot/meshes/my_spider/sr1.STL
- link rear_right_link0: geometry collision mesh filename=package://spiderbot/meshes/my_spider/r1.STL; visual mesh filename=package://spiderbot/meshes/my_spider/r1.STL
- link rear_right_link1: geometry collision mesh filename=package://spiderbot/meshes/my_spider/sr1.STL; visual mesh filename=package://spiderbot/meshes/my_spider/sr1.STL

File: quadruped_spider/spiderbot/urdf/spiderbot.xacro (robot description, xacro)
@@ -23,6 +23,6 @@
 						<samples>720</samples>
 						<resolution>1</resolution>
-						<min_angle>-1.570796</min_angle>
-              			<max_angle>1.570796</max_angle>
+						<min_angle>-3.1415926536</min_angle>
+              			<max_angle>3.1415926536</max_angle>
               		</horizontal>
               	</scan>
@@ -94,5 +94,5 @@
 </gazebo>
  <joint type="fixed" name="camera_joint">
-   <origin xyz="0.05 0 0.12" rpy="0 0 0"/>
+   <origin xyz="0 -0.05 0.05" rpy="0 0 -1.5708"/>
    <child link="camera"/>
    <parent link="base_link"/>
@@ -173,9 +173,9 @@
 	</gazebo>
     <!--Dummy Link-->
-    <link name="dummy_link">
+    <!-- <link name="dummy_link">
 	</link>
 	<joint name="dummy_joint" type="fixed">
 		<parent link="dummy_link"/>
 		<child link="base_link"/>
-	</joint>
+	</joint> -->
 </robot>
